File: Modbus_IO_Board.sch (KiCad schematic (older format))
At the start: 68 parts, among them IC1 ATMEGA328PB-AN, IC2 TPS7B6933QDCYRQ1, IC3 MAX3072EASA+, IC4 SN74LVC2G14DBVRG4, IC5 LTV-206, J1 Conn_01x06_Male, J2 282834-5, J3 282834-5, U1 PSM712-LF-T7, Y1 7.37MHz

Commit message: PCB awaiting Review
Parts:
- J2: value 282834-5 -> 2.54mm pitch Terminal Block
Connections:
- net 1Y: now also IC1.23 (PC0_(ADC0/PTCY/MISO1)); no longer IC1.10 ((OC0A/PTCXY/AIN0)_PD6)
- net 2Y: now also IC1.24 (PC1_(ADC1/PTCY/SCK1)); no longer IC1.11 ((PTCXY/AIN1)_PD7)
- net OUT1: now also IC1.32 (PD2_(PTCXY/INT0/OC3B/OC4B)); no longer IC1.12 ((ICP1/CLKO/PTCXY)_PB0)
- net OUT2: now also IC1.1 ((OC2B/INT1/PTCXY)_PD3); no longer IC1.13 ((OC1A/PTCXY)_PB1)
- net 1A: no longer names the net of C13.1, D6.2, D7.1 (A1), IC4.1 (1A), R6.2
- net 2A: no longer names the net of C14.1, D8.2, D9.1 (A1), IC4.3 (2A), R8.2
Other:
- note added: "Pin 5 for wire shielding \nground if present"
- moved on the sheet: C13, D6, D7, R6

Commit message: Review Pending
Parts:
- C10: value 4.7uF10V -> 4.7uF
- D10, D11: footprint Diode_SMD:D_MELF -> Diode_SMD:D_SOD-323
Changed lines of the file:
@@
 AR Path="/6152DE2D/6154F36E" Ref="C?"  Part="1"
 F 0 "C10" V 15679 7808 31  0000 L CNN
-F 1 "4.7uF10V" V 15479 7758 31  0000 L CNN
+F 1 "4.7uF" V 15479 7758 31  0000 L CNN
 F 2 "Capacitor_SMD:C_1206_3216Metric" H 15579 7858 50  0001 C CNN
 F 3 "~" H 15579 7858 50  0001 C CNN
@@
 F 0 "D11" V 8220 5010 50  0000 L CNN
 F 1 "D_TVS" H 8330 4960 50  0000 L CNN
-F 2 "Diode_SMD:D_MELF" H 8440 5050 50  0001 C CNN
+F 2 "Diode_SMD:D_SOD-323" H 8440 5050 50  0001 C CNN
 F 3 "~" H 8440 5050 50  0001 C CNN
 	1    8440 5050
@@
 F 0 "D10" V 8640 5400 50  0000 L CNN
 F 1 "D_TVS" H 8320 5360 50  0000 L CNN
-F 2 "Diode_SMD:D_MELF" H 8430 5450 50  0001 C CNN
+F 2 "Diode_SMD:D_SOD-323" H 8430 5450 50  0001 C CNN
 F 3 "~" H 8430 5450 50  0001 C CNN
 	1    8430 5450
