File: Modbus_IO_Board.kicad_pcb (KiCad board)
At the start: 2 copper layers, 71.5 x 45 mm, 74 parts, among them IC1 ATMEGA328PB-AN, IC2 TPS7B6933QDCYRQ1, IC3 MAX3072EASA+, IC4 SN74LVC2G14DBVRG4, IC5 LTV-206, J1 Conn_01x06_Male, J2 282834-5, J3 282834-5, U1 PSM712-LF-T7, Y1 7.37MHz

Commit message: PCB awaiting Review
Parts:
- moved G*** 184.4 mm to (228.5, 102.5)
- moved G*** 96.9 mm to (163.0, 102.5)
- moved D4 46.1 mm to (190.2, 112.5)
- moved C10 46.0 mm to (184.2, 100.5)
- moved RV1 46.0 mm to (185.0, 113.3)
- moved IC2 45.8 mm to (185.5, 106.1)
- moved RT1 43.5 mm to (179.7, 109.4)
- moved C8 42.6 mm to (189.2, 99.2), turned to 0 degrees
- moved C9 41.7 mm to (190.3, 103.5), turned to 90 degrees
- moved D3 41.2 mm to (180.4, 111.8)
- moved FB1 40.5 mm to (190.3, 108.3)
- moved IC5 24.9 mm to (217.7, 98.9)
- moved D8 23.9 mm to (176.1, 94.9), turned to 90 degrees
- moved R5 23.8 mm to (217.8, 94.5), turned to 0 degrees
- moved R4 23.7 mm to (215.3, 94.5), turned to 0 degrees
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- renumbered TP16 to 12V, TP12 to 12V, TP9 to A, TP13 to A, TP10 to B, TP14 to B, TP3 to EN, TP15 to GND, TP11 to GND, TP6 to GND, TP5 to GND, TP4 to GND, TP1 to RX
Connections:
- IC1 pad 1: Net-(IC1-Pad1) -> /OUT2
- IC1 pad 10: /1Y -> Net-(IC1-Pad10)
- IC1 pad 11: /2Y -> Net-(IC1-Pad11)
- IC1 pad 12: /OUT1 -> Net-(IC1-Pad12)
- IC1 pad 13: /OUT2 -> Net-(IC1-Pad13)
- IC1 pad 23: Net-(IC1-Pad23) -> /1Y
- IC1 pad 24: Net-(IC1-Pad24) -> /2Y
- IC1 pad 32: Net-(IC1-Pad32) -> /OUT1
Routing:
- net +3V3: track 9.55 -> 96.3 mm, vias 0 -> 3
- net GND: track 4.35 -> 80.5 mm, vias 0 -> 38
- net Net-(D10-Pad1): track 0.00 -> 58.3 mm, vias 0 -> 2
- net Net-(D11-Pad2): track 0.00 -> 58.1 mm, vias 0 -> 2
- net /I2-1: track 0.00 -> 56.5 mm, vias 0 -> 1
- net /I1-1: track 0.00 -> 46.1 mm
- net +12V: track 0.00 -> 45.8 mm
- net Net-(D11-Pad1): track 0.00 -> 44.3 mm
- net /Data_A: track 6.56 -> 47.3 mm
- net /Data_B: track 6.31 -> 44.2 mm
- net Net-(D10-Pad2): track 0.00 -> 34.1 mm
- net /OUT1: track 0.00 -> 20.5 mm, vias 0 -> 2
- net /OUT2: track 0.00 -> 19.4 mm, vias 0 -> 2
- net Net-(C8-Pad1): track 0.00 -> 15.5 mm
- net /1Y: track 0.00 -> 15.4 mm, vias 0 -> 2
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- added copper zone on B.Cu, net GND
Other:
- outline, holes or cut-outs redrawn
- board text added: "12V"
- board text added: "3.3V"
- board text added: "GND"
- board text added: "I1.1"
- board text added: "I1.2"
- board text added: "I2.1"
- board text added: "I2.2"
- board text added: "MADE IN INDIA"
- board text added: "MISO"
- board text added: "MOSI"
- board text added: "O1.1"
- board text added: "O1.2"
- board text added: "O2.1"
- board text added: "O2.2"
- board text added: "RSB"
- board text added: "SCK"

Commit message: Review Pending
Parts:
- C10: value 4.7uF10V -> 4.7uF
- D10, D11: footprint Diode_SMD:D_MELF -> Diode_SMD:D_SOD-323
- J2: value 282834-5 -> 2.54mm pitch Terminal Block
- moved D10 1.60 mm to (202.7, 115.1)
- moved G*** 1.12 mm to (228.3, 103.6)
- moved D11 0.74 mm to (208.1, 115.0)
- moved G*** 0.50 mm to (163.0, 103.0)
- renumbered RX to TP1, EN to TP3
Connections:
- net /1A renamed Net-(C13-Pad1)
- net /2A renamed Net-(C14-Pad1)
- B pad 1: (no net) -> /Data_B
Routing:
- net GND: track 80.5 -> 86.0 mm
- net Net-(D10-Pad2): track 34.1 -> 30.1 mm
- net Net-(D10-Pad1): track 58.3 -> 56.0 mm
- net Net-(D11-Pad2): track 58.1 -> 57.2 mm
- net +3V3: track 96.3 -> 95.6 mm
Other:
- outline, holes or cut-outs redrawn

Commit message: Review and Approval Pending
Parts:
- moved G*** 0.71 mm to (228.8, 103.1)
- moved G*** 0.29 mm to (162.7, 103.1)
Routing:
- net GND: track 86.0 -> 82.8 mm, vias 38 -> 37
- net +3V3: track 95.6 -> 94.9 mm
Changed lines of the file:
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@@
     (thickness 1.6)
     (drawings 71)
-    (tracks 456)
+    (tracks 454)
     (zones 0)
     (modules 74)
@@
   )
   (module logo:A1_logo locked (layer F.Cu)
-    (at 228.3 103.6)
+    (at 228.8 103.1)
     (fp_text reference G*** (at 0.6096 -0.2794) (layer F.SilkS) hide
       (effects (font (size 0.8 0.8) (thickness 0.1)))
@@
   )
   (module logo:A1_logo locked (layer F.Cu)
-    (at 162.975 103)
+    (at 162.7 103.1)
     (fp_text reference G*** (at 0.375 -0.25) (layer F.SilkS) hide
       (effects (font (size 0.8 0.8) (thickness 0.1)))
@@
   (segment (start 170.22 105.03) (end 170.2 105.01) (width 0.8) (layer F.Cu) (net 1))
   (segment (start 170.22 110.24) (end 170.22 105.03) (width 0.8) (layer F.Cu) (net 1))
-  (segment (start 184.8 97.7) (end 185.4 97.7) (width 0.5) (layer F.Cu) (net 1))
-  (via (at 184.8 97.7) (size 0.8) (drill 0.4) (layers F.Cu B.Cu) (net 1))
-  (via (at 187.2 95.9) (size 0.8) (drill 0.4) (layers F.Cu B.Cu) (net 1))
-  (segment (start 185.4 97.7) (end 187.2 95.9) (width 0.5) (layer F.Cu) (net 1))
+  (segment (start 190.8 100.9) (end 190.8 100.9) (width 0.5) (layer F.Cu) (net 1))
+  (via (at 190.8 100.9) (size 0.8) (drill 0.4) (layers F.Cu B.Cu) (net 1))
   (segment (start 195.91 100.27) (end 196.19 100.27) (width 0.25) (layer F.Cu) (net 2))
   (segment (start 196.74 100.82) (end 197.52 100.82) (width 0.25) (layer F.Cu) (net 2))
@@
   (segment (start 202.075 93.3) (end 203.66 93.3) (width 0.5) (layer F.Cu) (net 3))
   (via (at 202.075 93.3) (size 0.8) (drill 0.4) (layers F.Cu B.Cu) (net 3))
-  (segment (start 193.875 99.725) (end 200.3 93.3) (width 0.5) (layer B.Cu) (net 3))
-  (segment (start 191.1 101.8) (end 185.3 96) (width 0.5) (layer B.Cu) (net 3))
-  (segment (start 193.875 101.8) (end 191.1 101.8) (width 0.5) (layer B.Cu) (net 3))
-  (segment (start 193.875 101.8) (end 193.875 99.725) (width 0.5) (layer B.Cu) (net 3))
   (segment (start 193.51 101.8) (end 192.77 102.54) (width 0.5) (layer F.Cu) (net 3))
-  (segment (start 185.3 96) (end 185.3 94.7) (width 0.5) (layer B.Cu) (net 3))
   (segment (start 193.875 101.8) (end 193.51 101.8) (width 0.5) (layer F.Cu) (net 3))
-  (segment (start 200.3 93.3) (end 202.075 93.3) (width 0.5) (layer B.Cu) (net 3))
   (via (at 193.875 101.8) (size 0.8) (drill 0.4) (layers F.Cu B.Cu) (net 3))
   (segment (start 213.5 97.6) (end 217.31 97.6) (width 0.5) (layer F.Cu) (net 3))
@@
   (segment (start 217.045 97.335) (end 217.31 97.6) (width 0.5) (layer F.Cu) (net 3))
   (segment (start 217.045 96.148) (end 217.045 97.335) (width 0.5) (layer F.Cu) (net 3))
+  (segment (start 186.7 94.7) (end 185.3 94.7) (width 0.5) (layer B.Cu) (net 3))
+  (segment (start 193.8 101.8) (end 186.7 94.7) (width 0.5) (layer B.Cu) (net 3))
+  (segment (start 193.875 101.8) (end 193.8 101.8) (width 0.5) (layer B.Cu) (net 3))
+  (segment (start 200.3 93.3) (end 202.075 93.3) (width 0.5) (layer B.Cu) (net 3))
+  (segment (start 193.875 99.725) (end 200.3 93.3) (width 0.5) (layer B.Cu) (net 3))
+  (segment (start 193.875 101.8) (end 193.875 99.725) (width 0.5) (layer B.Cu) (net 3))
   (segment (start 192.76 92.49) (end 195.17 92.49) (width 0.25) (layer F.Cu) (net 4))
   (segment (start 192.7 88.805) (end 192.705 88.8) (width 0.25) (layer F.Cu) (net 5))

Commit message: Review Pending
Parts:
- renumbered TP3 to EN, TP1 to RX
Changed lines of the file:
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@@
     (32 B.Adhes user)
     (33 F.Adhes user)
-    (34 B.Paste user)
+    (34 B.Paste user hide)
     (35 F.Paste user)
     (36 B.SilkS user)
@@
     (visible_elements 7FFDFFFF)
     (pcbplotparams
-      (layerselection 0x00030_7ffffffe)
+      (layerselection 0x3ffff_ffffffff)
       (usegerberextensions false)
       (usegerberattributes true)
@@
       (padsonsilk false)
       (subtractmaskfromsilk false)
-      (outputformat 3)
+      (outputformat 1)
       (mirror false)
       (drillshape 0)
@@
     (tags "test point SMD pad")
     (attr virtual)
-    (fp_text reference TP1 (at -0.13 -0.66) (layer F.SilkS)
+    (fp_text reference RX (at -0.13 -0.66) (layer F.SilkS)
       (effects (font (size 0.8 0.8) (thickness 0.1)))
     )
@@
       (effects (font (size 1 1) (thickness 0.15)))
     )
-    (fp_text user TX (at -0.8 -0.0592) (layer F.SilkS)
+    (fp_text user TX (at -0.6 0.0408) (layer F.SilkS)
       (effects (font (size 0.8 0.8) (thickness 0.1)))
     )
@@
     (tags capacitor)
     (attr smd)
-    (fp_text reference C1 (at 1.44 -0.42 180) (layer F.SilkS)
+    (fp_text reference C1 (at 1.44 -0.22 180) (layer F.SilkS)
       (effects (font (size 0.8 0.8) (thickness 0.1)))
     )
@@
     (tags "test point SMD pad")
     (attr virtual)
-    (fp_text reference TP3 (at -0.5 -0.98 180) (layer F.SilkS)
-      (effects (font (size 0.8 0.8) (thickness 0.1)))
-    )
+    (fp_text reference EN (at -0.5 -0.98 180) (layer F.SilkS)
+      (effects (font (size 0.8 0.8) (thickness 0.1)))
+    )
